File: mosquito-c3.kicad_sch (KiCad schematic)
At the start: 39 parts, among them J1 RJ12, J2 USB_C_Receptacle_USB2.0, Q1 MMBT3906T, SW1 SW_Push, SW2 SW_Push, U1 ESP32-C3-MINI-1, U2 TP6841S6

Commit message: pcb cleanup
Parts:
- D1: footprint Diode_SMD:D_SOD-123 -> mosquito:D_SOD-123
- D2, D3, D4, D5, D6: footprint Diode_SMD:D_SOD-523 -> mosquito:D_SOD-523
- Q1: footprint Package_TO_SOT_SMD:SOT-523 -> mosquito:SOT-523
Changed lines of the file:
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@@
       (effects (font (size 1.27 1.27)))
     )
-    (property "Footprint" "Diode_SMD:D_SOD-523" (at 115.57 81.28 0)
+    (property "Footprint" "mosquito:D_SOD-523" (at 115.57 81.28 0)
       (effects (font (size 1.27 1.27)) hide)
     )
@@
       (effects (font (size 1.27 1.27)) (justify left))
     )
-    (property "Footprint" "Package_TO_SOT_SMD:SOT-523" (at 135.89 84.455 0)
+    (property "Footprint" "mosquito:SOT-523" (at 135.89 84.455 0)
       (effects (font (size 1.27 1.27) italic) (justify left) hide)
     )
@@
       (effects (font (size 1.27 1.27)))
     )
-    (property "Footprint" "Diode_SMD:D_SOD-523" (at 54.61 151.13 0)
+    (property "Footprint" "mosquito:D_SOD-523" (at 54.61 151.13 0)
       (effects (font (size 1.27 1.27)) hide)
     )
@@
       (effects (font (size 1.27 1.27)))
     )
-    (property "Footprint" "Diode_SMD:D_SOD-523" (at 54.61 140.97 0)
+    (property "Footprint" "mosquito:D_SOD-523" (at 54.61 140.97 0)
       (effects (font (size 1.27 1.27)) hide)
     )
@@
       (effects (font (size 1.27 1.27)))
     )
-    (property "Footprint" "Diode_SMD:D_SOD-523" (at 121.92 158.75 0)
+    (property "Footprint" "mosquito:D_SOD-523" (at 121.92 158.75 0)
       (effects (font (size 1.27 1.27)) hide)
     )
@@
       (effects (font (size 1.27 1.27)))
     )
-    (property "Footprint" "Diode_SMD:D_SOD-523" (at 124.46 76.2 0)
+    (property "Footprint" "mosquito:D_SOD-523" (at 124.46 76.2 0)
       (effects (font (size 1.27 1.27)) hide)
     )
@@
       (effects (font (size 1.27 1.27)))
     )
-    (property "Footprint" "Diode_SMD:D_SOD-123" (at 46.355 154.94 0)
+    (property "Footprint" "mosquito:D_SOD-123" (at 46.355 154.94 0)
       (effects (font (size 1.27 1.27) italic) (justify left) hide)
     )
