File: mosquito-c3.kicad_pcb (KiCad board)
At the start: 4 copper layers, 19.5 x 31 mm, 39 parts, among them J1 RJ12, J2 USB_C_Receptacle_USB2.0, Q1 MMBT3906T, SW1 SW_Push, SW2 SW_Push, U1 ESP32-C3-MINI-1, U2 TP6841S6

Commit message: pcb cleanup
Parts:
- D1: footprint Diode_SMD:D_SOD-123 -> mosquito:D_SOD-123
- D2: renamed from D3; footprint Diode_SMD:D_SOD-523 -> mosquito:D_SOD-523
- D3: renamed from D2; footprint Diode_SMD:D_SOD-523 -> mosquito:D_SOD-523
- D4, D5, D6: footprint Diode_SMD:D_SOD-523 -> mosquito:D_SOD-523
- Q1: footprint Package_TO_SOT_SMD:SOT-523 -> mosquito:SOT-523
- moved Q1 0.14 mm to (89.8, 45.0), turned to 90 degrees
- moved R8 0.14 mm to (89.7, 43.4)
- moved R9 0.13 mm to (89.7, 42.4)
Connections:
- D2 pad 2: Net-(D3-A) -> /USB_VBUS
- D3 pad 2: /USB_VBUS -> Net-(D3-A)
Routing:
- net Net-(D2-K): track 26.5 -> 31.8 mm
- net /USB_VBUS: track 57.0 -> 62.1 mm
- net +3V3: track 47.1 -> 49.9 mm
- net Net-(Q1-B): track 4.07 -> 1.32 mm
- net Net-(Q1-C): track 2.93 -> 1.14 mm
- net Net-(D3-A): track 1.63 -> 2.23 mm
- net /MBUS+: track 22.9 -> 23.5 mm

Commit message: add KiKit tab/panel hints
Parts:
- added REF**: Tab, PCM_kikit:Tab, F.Cu at (82.1, 33.4)
- added REF**: Tab, PCM_kikit:Tab, F.Cu at (84.7, 65.5)
Changed lines of the file:
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@@
       (drillshape 0)
       (scaleselection 1)
-      (outputdirectory "gerber-c3/")
+      (outputdirectory "gerber/")
     )
   )
@@
     )
   )
+  (footprint "PCM_kikit:Tab" (layer "F.Cu")
+    (at 82.1 33.4 -90)
+    (descr "A symbol representing annotation for tab placement")
+    (attr exclude_from_pos_files exclude_from_bom)
+    (fp_text reference "REF**" (at 0 -2 90) (layer "F.SilkS") hide
+        (effects (font (size 1 1) (thickness 0.15)))
+    )
+    (fp_text value "Tab" (at -2.75 -1 90) (layer "Dwgs.User")
+        (effects (font (size 1.2 1.2) (thickness 0.2)))
+    )
+    (fp_text user "KIKIT: width: 10mm" (at -5.5 0) (layer "Dwgs.User")
+        (effects (font (size 1 1) (thickness 0.15)))
+    )
+    (fp_line (start 0.25 0) (end -2.75 0)
+      (stroke (width 0.3) (type solid)) (layer "Dwgs.User"))
+    (fp_line (start 0.25 0) (end -0.75 -1)
+      (stroke (width 0.3) (type solid)) (layer "Dwgs.User"))
+    (fp_line (start 0.25 0) (end -0.75 1)
+      (stroke (width 0.3) (type solid)) (layer "Dwgs.User"))
+    (fp_line (start 0.25 1) (end 0.25 -1)
+      (stroke (width 0.3) (type solid)) (layer "Dwgs.User"))
+  )
   (footprint "Resistor_SMD:R_0402_1005Metric" (layer "F.Cu")
     (at 84.15 49.84 90)
@@
     )
   )
+  (footprint "PCM_kikit:Tab" (layer "F.Cu")
+    (at 84.7 65.5 90)
+    (descr "A symbol representing annotation for tab placement")
+    (attr exclude_from_pos_files exclude_from_bom)
+    (fp_text reference "REF**" (at 0 -2 90) (layer "F.SilkS") hide
+        (effects (font (size 1 1) (thickness 0.15)))
+    )
+    (fp_text value "Tab" (at -2.75 -1 90) (layer "Dwgs.User")
+        (effects (font (size 1.2 1.2) (thickness 0.2)))
+    )
+    (fp_text user "KIKIT: width: 14mm" (at -5.5 0) (layer "Dwgs.User")
+        (effects (font (size 1 1) (thickness 0.15)))
+    )
+    (fp_line (start 0.25 0) (end -2.75 0)
+      (stroke (width 0.3) (type solid)) (layer "Dwgs.User"))
+    (fp_line (start 0.25 0) (end -0.75 -1)
+      (stroke (width 0.3) (type solid)) (layer "Dwgs.User"))
+    (fp_line (start 0.25 0) (end -0.75 1)
+      (stroke (width 0.3) (type solid)) (layer "Dwgs.User"))
+    (fp_line (start 0.25 1) (end 0.25 -1)
+      (stroke (width 0.3) (type solid)) (layer "Dwgs.User"))
+  )
   (footprint "mosquito:LED_0404" (layer "F.Cu")
